Commit message: revise urdf files

File: irb6640_185_280_or.urdf (robot description, URDF)
Before this commit: robot abb_irb6640_185_280, 12 links, 11 joints
Links:
- link vacuum_gripper: geometry collision mesh filename=package://irb6640_gazebo/models/vacuum_gripper.stl scale=1.254 1.254 1.254; visual mesh filename=package://irb6640_gazebo/models/vacuum_gripper.stl scale=1.254 1.254 1.254
Joints:
- joint joint_6: origin xyz=0.15 0 0 rpy=0 0 0 -> xyz=0.2 0 0 rpy=0 0 0
- joint link_6_vacuum_gripper: origin xyz=0.25 0 0 rpy=0 -1.57079632679 0 -> xyz=0.15 0 0 rpy=0 -1.57079632679 0

File: testbed.urdf (robot description, URDF)
Before this commit: robot wall, 2 links, 1 joints
Joints:
- joint joint: origin xyz=1.0 -0.94 0.32 rpy=0 0 -1.57 -> xyz=4.0 3.0 0 rpy=0 0 -1.57

Commit message: adjust vacuum gripper orientation

File: irb6640_185_280_or.urdf (robot description, URDF)
Before this commit: robot abb_irb6640_185_280, 12 links, 11 joints
Joints:
- joint joint_6-panel: origin xyz=0.2 0 -0.2 rpy=1.57079632679 0 -1.57079632679 -> xyz=0.1 0 -0.2 rpy=1.57079632679 0 -1.57079632679
- joint link_6_vacuum_gripper: origin xyz=0.15 0 0 rpy=0 -1.57079632679 0 -> xyz=0.15 0 0 rpy=-1.57079632679 0 1.57079632679
